File: v0.2/boards/cm_ltc6102/cm_ltc6102.sch (EAGLE design)
At the start: 93 parts, among them J1 10118194-0001LF, U1 ADA4528-2ARMZ-R7, U10 TS5A3159ADBVRDBV6-M, U2 LTC6102IMS8PBF, U3 ADM7170ACPZ-1.3-R7CP_8_21-M, U4 MIC2250-1YD5TSOT-23-5_D5-M, U5 INA226_DGS_10DGS10-M, U6 TS3A4751PWRPW14-M, U7 TS5A4624DCKRDCK6-M, X1 PN87520-S

Commit message: cm_ltc6102: add dgnd and agnd connection, fix silk-screen
Parts:
- added SH1: SHORT-VT5, shorts-old:SHORT-VT5
- added TP10, TP11, TP3, TP4, TP5: TPTP11R, testpad:TPTP11R
Connections:
- net ADA_VCC: now also TP4.TP
- net DGND: now also SH1.P$2
- net GND: now also SH1.P$1
- net INA_VCC: now also TP5.TP
- net LTC_VCC: now also TP3.TP
- net SHUNT_V+: now also TP10.TP
- net SHUNT_V-: now also TP11.TP
Changed lines of the file:
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@@
 <part name="TP8" library="testpad" library_urn="urn:adsk.eagle:library:385" deviceset="TP" device="TP11R" package3d_urn="urn:adsk.eagle:package:27961/1"/>
 <part name="TP9" library="testpad" library_urn="urn:adsk.eagle:library:385" deviceset="TP" device="TP11R" package3d_urn="urn:adsk.eagle:package:27961/1"/>
+<part name="TP3" library="testpad" library_urn="urn:adsk.eagle:library:385" deviceset="TP" device="TP11R" package3d_urn="urn:adsk.eagle:package:27961/1"/>
+<part name="TP4" library="testpad" library_urn="urn:adsk.eagle:library:385" deviceset="TP" device="TP11R" package3d_urn="urn:adsk.eagle:package:27961/1"/>
+<part name="TP5" library="testpad" library_urn="urn:adsk.eagle:library:385" deviceset="TP" device="TP11R" package3d_urn="urn:adsk.eagle:package:27961/1"/>
+<part name="TP10" library="testpad" library_urn="urn:adsk.eagle:library:385" deviceset="TP" device="TP11R" package3d_urn="urn:adsk.eagle:package:27961/1"/>
+<part name="TP11" library="testpad" library_urn="urn:adsk.eagle:library:385" deviceset="TP" device="TP11R" package3d_urn="urn:adsk.eagle:package:27961/1"/>
+<part name="SH1" library="shorts-old" deviceset="SHORT-V" device="T5"/>
 </parts>
 <sheets>
@@
 <instance part="TP8" gate="G$1" x="-256.54" y="91.44"/>
 <instance part="TP9" gate="G$1" x="-256.54" y="177.8"/>
+<instance part="TP3" gate="G$1" x="-144.78" y="330.2"/>
+<instance part="TP4" gate="G$1" x="-144.78" y="297.18"/>
+<instance part="TP5" gate="G$1" x="-144.78" y="363.22"/>
+<instance part="TP10" gate="G$1" x="68.58" y="365.76"/>
+<instance part="TP11" gate="G$1" x="111.76" y="365.76"/>
+<instance part="SH1" gate="G$1" x="-241.3" y="299.72" rot="R90"/>
 </instances>
 <busses>
@@
 <net name="SHUNT_V-" class="0">
 <segment>
-<wire x1="96.52" y1="363.22" x2="119.38" y2="363.22" width="0.1524" layer="91"/>
+<wire x1="96.52" y1="363.22" x2="111.76" y2="363.22" width="0.1524" layer="91"/>
 <pinref part="U$1" gate="A" pin="I2"/>
 <label x="121.92" y="363.22" size="1.778" layer="95"/>
+<pinref part="TP11" gate="G$1" pin="TP"/>
+<wire x1="111.76" y1="363.22" x2="119.38" y2="363.22" width="0.1524" layer="91"/>
+<junction x="111.76" y="363.22"/>
 </segment>
 <segment>
@@
 <pinref part="U$1" gate="A" pin="I1"/>
 <label x="50.8" y="363.22" size="1.778" layer="95"/>
-<wire x1="55.88" y1="363.22" x2="81.28" y2="363.22" width="0.1524" layer="91"/>
+<wire x1="55.88" y1="363.22" x2="68.58" y2="363.22" width="0.1524" layer="91"/>
+<pinref part="TP10" gate="G$1" pin="TP"/>
+<wire x1="68.58" y1="363.22" x2="81.28" y2="363.22" width="0.1524" layer="91"/>
+<junction x="68.58" y="363.22"/>
 </segment>
 <segment>
@@
 <wire x1="-144.78" y1="327.66" x2="-142.24" y2="327.66" width="0.1524" layer="91"/>
 <label x="-147.32" y="327.66" size="1.778" layer="95" rot="R180"/>
+<pinref part="TP3" gate="G$1" pin="TP"/>
+<junction x="-144.78" y="327.66"/>
 </segment>
 </net>
@@
 <wire x1="-48.26" y1="124.46" x2="-48.26" y2="114.3" width="0.1524" layer="91"/>
 <pinref part="GND16" gate="1" pin="GND"/>
+</segment>
+<segment>
+<pinref part="GND35" gate="1" pin="GND"/>
+<wire x1="-231.14" y1="299.72" x2="-231.14" y2="294.64" width="0.1524" layer="91"/>
+<pinref part="SH1" gate="G$1" pin="P$1"/>
+<wire x1="-238.76" y1="299.72" x2="-231.14" y2="299.72" width="0.1524" layer="91"/>
 </segment>
 </net>
@@
 <wire x1="-144.78" y1="294.64" x2="-142.24" y2="294.64" width="0.1524" layer="91"/>
 <label x="-147.32" y="294.64" size="1.778" layer="95" rot="R180"/>
+<pinref part="TP4" gate="G$1" pin="TP"/>
+<junction x="-144.78" y="294.64"/>
 </segment>
 </net>
@@
 <pinref part="R19" gate="G$1" pin="1"/>
 <wire x1="-142.24" y1="360.68" x2="-144.78" y2="360.68" width="0.1524" layer="91"/>
+<pinref part="TP5" gate="G$1" pin="TP"/>
+<junction x="-144.78" y="360.68"/>
 </segment>
 <segment>
@@
 <pinref part="SUPPLY2" gate="G$1" pin="DGND"/>
 <wire x1="-248.92" y1="294.64" x2="-248.92" y2="299.72" width="0.1524" layer="91"/>
-<wire x1="-248.92" y1="299.72" x2="-248.92" y2="304.8" width="0.1524" layer="91"/>
-<junction x="-248.92" y="299.72"/>
 <wire x1="-248.92" y1="299.72" x2="-259.08" y2="299.72" width="0.1524" layer="91"/>
 <label x="-269.24" y="299.72" size="1.778" layer="95"/>
-<pinref part="GND35" gate="1" pin="GND"/>
-<wire x1="-231.14" y1="304.8" x2="-231.14" y2="299.72" width="0.1524" layer="91"/>
-<wire x1="-231.14" y1="299.72" x2="-231.14" y2="294.64" width="0.1524" layer="91"/>
-<junction x="-231.14" y="299.72"/>
-<wire x1="-248.92" y1="304.8" x2="-231.14" y2="304.8" width="0.1524" layer="91"/>
-<wire x1="-231.14" y1="299.72" x2="-248.92" y2="299.72" width="0.1524" layer="91"/>
-</segment>
-<segment>
+<pinref part="SH1" gate="G$1" pin="P$2"/>
+<wire x1="-243.84" y1="299.72" x2="-248.92" y2="299.72" width="0.1524" layer="91"/>
+</segment>
+<segment>

Commit message: fix some missing gnd wires
Connections:
- removed net LTC_OUT: C2.1, R11.2
- removed net N$4: R27.2, R28.2
- net 5V: no longer U3.SENSE
- net 5V_R: now also U3.SENSE
- net GND: now also R27.2, R28.2
- net S1_OUT: now also C2.1, R11.2
Changed lines of the file:
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@@
 <wire x1="-238.76" y1="299.72" x2="-231.14" y2="299.72" width="0.1524" layer="91"/>
+</segment>
+<segment>
+<pinref part="R28" gate="G$1" pin="2"/>
+<wire x1="-256.54" y1="66.04" x2="-256.54" y2="60.96" width="0.1524" layer="91"/>
+<pinref part="GND30" gate="1" pin="GND"/>
+</segment>
+<segment>
+<pinref part="R27" gate="G$1" pin="2"/>
+<wire x1="-208.28" y1="149.86" x2="-208.28" y2="147.32" width="0.1524" layer="91"/>
+<pinref part="GND29" gate="1" pin="GND"/>
 </segment>
 </net>
@@
 <wire x1="53.34" y1="426.72" x2="53.34" y2="416.56" width="0.1524" layer="91"/>
 <wire x1="53.34" y1="416.56" x2="71.12" y2="416.56" width="0.1524" layer="91"/>
-</segment>
-</net>
-<net name="LTC_OUT" class="0">
-<segment>
-<wire x1="256.54" y1="431.8" x2="256.54" y2="426.72" width="0.1524" layer="91"/>
-<pinref part="C2" gate="G$1" pin="1"/>
-<pinref part="R11" gate="G$1" pin="2"/>
-<wire x1="256.54" y1="431.8" x2="264.16" y2="431.8" width="0.1524" layer="91"/>
 </segment>
 </net>
@@
 <wire x1="304.8" y1="317.5" x2="304.8" y2="312.42" width="0.1524" layer="91"/>
 <label x="358.14" y="317.5" size="1.778" layer="95"/>
+<junction x="304.8" y="312.42"/>
 </segment>
 <segment>
@@
 </segment>
 </net>
-<net name="5V" class="0">
-<segment>
-<pinref part="U3" gate="A" pin="SENSE"/>
-<wire x1="-165.1" y1="81.28" x2="-160.02" y2="81.28" width="0.1524" layer="91"/>
-<label x="-157.48" y="81.28" size="1.778" layer="95"/>
-</segment>
-<segment>
-<wire x1="-111.76" y1="327.66" x2="-104.14" y2="327.66" width="0.1524" layer="91"/>
-<label x="-101.6" y="327.66" size="1.778" layer="95"/>
-<pinref part="L3" gate="A" pin="1"/>
-</segment>
-<segment>
-<wire x1="-111.76" y1="294.64" x2="-104.14" y2="294.64" width="0.1524" layer="91"/>
-<label x="-101.6" y="294.64" size="1.778" layer="95"/>
-<pinref part="L2" gate="A" pin="1"/>
-</segment>
-<segment>
-<wire x1="-111.76" y1="360.68" x2="-104.14" y2="360.68" width="0.1524" layer="91"/>
-<label x="-101.6" y="360.68" size="1.778" layer="95"/>
-<pinref part="L5" gate="A" pin="1"/>
-</segment>
-<segment>
-<wire x1="-78.74" y1="86.36" x2="-86.36" y2="86.36" width="0.1524" layer="91"/>
-<label x="-93.98" y="86.36" size="1.778" layer="95"/>
-<pinref part="JMP1" gate="-0R" pin="2"/>
-</segment>
-</net>
 <net name="N$14" class="0">
 <segment>
@@
 <net name="S1_OUT" class="0">
 <segment>
+<pinref part="U2" gate="A" pin="OUT"/>
+<wire x1="71.12" y1="414.02" x2="53.34" y2="414.02" width="0.1524" layer="91"/>
+<label x="50.8" y="414.02" size="1.778" layer="95" rot="R180"/>
+</segment>
+<segment>
+<wire x1="256.54" y1="431.8" x2="256.54" y2="426.72" width="0.1524" layer="91"/>
+<pinref part="C2" gate="G$1" pin="1"/>
+<pinref part="R11" gate="G$1" pin="2"/>
+<wire x1="256.54" y1="431.8" x2="264.16" y2="431.8" width="0.1524" layer="91"/>
 <wire x1="248.92" y1="431.8" x2="248.92" y2="426.72" width="0.1524" layer="91"/>
 <pinref part="R10" gate="G$1" pin="2"/>
@@
 <junction x="248.92" y="431.8"/>
 <pinref part="TP1" gate="G$1" pin="TP"/>
-</segment>
-<segment>
-<pinref part="U2" gate="A" pin="OUT"/>
-<wire x1="71.12" y1="414.02" x2="53.34" y2="414.02" width="0.1524" layer="91"/>
-<label x="50.8" y="414.02" size="1.778" layer="95" rot="R180"/>
+<junction x="256.54" y="431.8"/>
 </segment>
 </net>
@@
 <pinref part="R27" gate="G$1" pin="1"/>
 <wire x1="-208.28" y1="162.56" x2="-208.28" y2="160.02" width="0.1524" layer="91"/>
-</segment>
-</net>
-<net name="N$4" class="0">
-<segment>
-<pinref part="R27" gate="G$1" pin="2"/>
-<wire x1="-208.28" y1="149.86" x2="-208.28" y2="147.32" width="0.1524" layer="91"/>
-<pinref part="GND29" gate="1" pin="GND"/>
-</segment>
-<segment>
-<pinref part="R28" gate="G$1" pin="2"/>
-<wire x1="-256.54" y1="66.04" x2="-256.54" y2="60.96" width="0.1524" layer="91"/>
-<pinref part="GND30" gate="1" pin="GND"/>
 </segment>
 </net>
@@
 <junction x="-256.54" y="88.9"/>
 </segment>
+<segment>
+<pinref part="U3" gate="A" pin="SENSE"/>
+<wire x1="-165.1" y1="81.28" x2="-160.02" y2="81.28" width="0.1524" layer="91"/>
+<label x="-157.48" y="81.28" size="1.778" layer="95"/>
+</segment>
 </net>
 <net name="5V_F" class="0">
@@
 </segment>
 </net>
+<net name="5V" class="0">
+<segment>
+<wire x1="-111.76" y1="360.68" x2="-104.14" y2="360.68" width="0.1524" layer="91"/>
+<label x="-101.6" y="360.68" size="1.778" layer="95"/>
+<pinref part="L5" gate="A" pin="1"/>
+</segment>
+<segment>
+<wire x1="-111.76" y1="327.66" x2="-104.14" y2="327.66" width="0.1524" layer="91"/>
+<label x="-101.6" y="327.66" size="1.778" layer="95"/>
+<pinref part="L3" gate="A" pin="1"/>
+</segment>
+<segment>
+<wire x1="-111.76" y1="294.64" x2="-104.14" y2="294.64" width="0.1524" layer="91"/>
+<label x="-101.6" y="294.64" size="1.778" layer="95"/>
+<pinref part="L2" gate="A" pin="1"/>
+</segment>
+<segment>
+<wire x1="-78.74" y1="86.36" x2="-86.36" y2="86.36" width="0.1524" layer="91"/>
+<label x="-93.98" y="86.36" size="1.778" layer="95"/>
+<pinref part="JMP1" gate="-0R" pin="2"/>
+</segment>
+</net>
