File: v0.2/board/cm_AD8629.sch (EAGLE design)
At the start: 81 parts, among them Q1 6.5A/20V/35mΩ, U2 LT8582EDKDPBF, U3 ADM7170ACPZ-1.3-R7CP_8_21-M, U4 MIC2250-1YD5TSOT-23-5_D5-M

Commit message: add usb entry
Parts:
- added J1: USB_A_SMT_FEMALE, SparkFun-Connectors:USB_A_SMT_FEMALE
Connections:
- new net N$15: J1.D+
- new net N$16: J1.D-
- net 5VUSB: now also J1.VBUS
- net GND: now also J1.GND
Changed lines of the file:
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@@
 <part name="SEL-SPLY1" library="SparkFun-Connectors" deviceset="CONN_02" device=""/>
 <part name="SUPPLY10" library="SparkFun-PowerSymbols" deviceset="VDD" device=""/>
+<part name="J1" library="SparkFun-Connectors" deviceset="USB_A" device="_SMT_FEMALE"/>
+<part name="GND33" library="supply1" library_urn="urn:adsk.eagle:library:371" deviceset="GND" device=""/>
 </parts>
 <sheets>
@@
 <instance part="SEL-SPLY1" gate="G$1" x="12.7" y="162.56"/>
 <instance part="SUPPLY10" gate="VDD" x="25.4" y="167.64"/>
+<instance part="J1" gate="G$1" x="71.12" y="132.08" rot="R180"/>
+<instance part="GND33" gate="1" x="91.44" y="132.08"/>
 </instances>
 <busses>
@@
 <pinref part="GND28" gate="1" pin="GND"/>
 <pinref part="R29" gate="G$1" pin="2"/>
+</segment>
+<segment>
+<pinref part="J1" gate="G$1" pin="GND"/>
+<pinref part="GND33" gate="1" pin="GND"/>
+<wire x1="78.74" y1="134.62" x2="91.44" y2="134.62" width="0.1524" layer="91"/>
 </segment>
 </net>
@@
 <label x="111.76" y="165.1" size="1.778" layer="95" xref="yes"/>
 </segment>
+<segment>
+<pinref part="J1" gate="G$1" pin="VBUS"/>
+<wire x1="78.74" y1="127" x2="81.28" y2="127" width="0.1524" layer="91"/>
+<label x="81.28" y="127" size="1.27" layer="95" xref="yes"/>
+</segment>
 </net>
 <net name="VSPLY1" class="0">
@@
 </segment>
 </net>
+<net name="N$15" class="0">
+<segment>
+<pinref part="J1" gate="G$1" pin="D+"/>
+<wire x1="78.74" y1="132.08" x2="81.28" y2="132.08" width="0.1524" layer="91"/>
+</segment>
+</net>
+<net name="N$16" class="0">
+<segment>
+<pinref part="J1" gate="G$1" pin="D-"/>
+<wire x1="78.74" y1="129.54" x2="81.28" y2="129.54" width="0.1524" layer="91"/>
+</segment>
+</net>

Commit message: first version of layout
add bom file

fix issues
Parts:
- removed CR1, CR2, CR3: 1N5818-B, 1N5818-B:1N5818-B
- removed U$6: SHUNT-RES, SparkFun-Resistors:SHUNT-RES
- removed U$9: 4.7u, SparkFun-Coils:1239AS-H
- removed U3: ADM7170ACPZ-1.3-R7CP_8_21-M, analog_devices:ADM7170ACPZ-1.3-R7CP_8_21-M
- removed U4: MIC2250-1YD5TSOT-23-5_D5-M, texas_instruments:MIC2250-1YD5TSOT-23-5_D5-M
- added BOOST: MIC2250-1YD5TSOT-23-5_D5-M, texas_instruments:MIC2250-1YD5TSOT-23-5_D5-M
- added C22: 1uF, SparkFun-Capacitors:10UF-0603-6.3V-20%
- added C23: 10uF, SparkFun-Capacitors:10UF-0603-6.3V-20%
- added CALIB-RES: (no value), pinhead:PINHD-1X4
- added CTRL: (no value), pinhead:PINHD-1X2
- added D1, D2, D3: 120mA/40V/370mV, SparkFun-DiscreteSemi:DIODE-SCHOTTKY-RB751S40
- added L1, L2, L5: 4.7u, SparkFun-Coils:1239AS-H
- added R33, R34: 1k, SparkFun-Resistors:150KOHM-0603-1/10W-1%
- added R35, R49, R51, R52, R53: 100k, SparkFun-Resistors:8.2KOHM-0603-1/10W-5%
- added R36: 0, SparkFun-Resistors:8.2KOHM-0603-1/10W-5%
- added R45, R46: 1k, SparkFun-Resistors:8.2KOHM-0603-1/10W-5%
- added R47: 10M, SparkFun-Resistors:8.2KOHM-0603-1/10W-5%
- added R48: 1M, SparkFun-Resistors:8.2KOHM-0603-1/10W-5%
- added R50: 10k, SparkFun-Resistors:8.2KOHM-0603-1/10W-5%
- added REG: ADM7170ACPZ-1.3-R7CP_8_21-M, analog_devices:ADM7170ACPZ-1.3-R7CP_8_21-M
- added SPLY-EXT: (no value), SparkFun-Connectors:CONN_02
- added TS5A23166_1, TS5A23166_2: TS5A23166DCURDCU8-M, texas_instruments:TS5A23166DCURDCU8-M
- added TS5A3159: TS5A3159ADBVRDBV6-M, texas_instruments:TS5A3159ADBVRDBV6-M
- added VCALIB_LED, VMCU_LED: (no value), led:LEDCHIPLED_0603
- C15: value 4700p -> 4.7uF
- C16: value 2200p -> 2.2uF
- R31, R32: value 1K 1% -> 100k; device rcl:R-US_R0603 -> SparkFun-Resistors:8.2KOHM-0603-1/10W-5%
- U$1: value 4.7u -> SHUNT-RES; device SparkFun-Coils:1239AS-H -> SparkFun-Resistors:SHUNT-RES
- renumbered AD8629 to AD8629-1, Q1 to MOSFET, U$2 to AD8629-2, U$3 to AD8629-3, U$4 to AD8629-4, U$5 to AD8422, U$7 to L3, U$8 to L4, U2 to +-12V
Connections:
- removed net 5V: +-12V.VC1, +-12V.VIN2, C10.1, L3.1, L4.1, R20.2, R21.2, R22.2, R23.2
- removed net N$25: MCU_VUSB.C, R31.1
- removed net N$26: R32.1, VMCU_EXT.C
- removed net VIN1: +-12V.VIN1
- removed net V_BATT: AD8422.IN+, R1.1
- removed net V_EXT: TS5A4624.NO, VMCU_EXT.A
- new net 5VIN: C22.1, J1.VBUS, L5.1
- new net 5V_F: TS5A3159.V+
- new net N$12: MCU_VUSB.C, R33.1
- new net N$19: R34.1, VMCU_EXT.C
- new net N$23: R45.2, VCALIB_LED.C
- new net N$24: R46.2, VMCU_LED.C
- new net N$30: R50.2, TS5A23166_1.COM1
- new net N$31: R49.2, TS5A23166_1.COM2
- new net N$32: R48.2, TS5A23166_2.COM1
- new net N$33: R47.2, TS5A23166_2.COM2
- new net SW_CTRL_0: CTRL.1, R52.2, TS5A3159.IN
- new net SW_CTRL_1: CALIB-RES.1, R53.2, TS5A23166_1.NO1
- new net SW_CTRL_2: CALIB-RES.2, R31.2, TS5A23166_1.NO2
- new net SW_CTRL_3: CALIB-RES.3, R32.2, TS5A23166_2.NO1
- new net SW_CTRL_4: CALIB-RES.4, R35.2, TS5A23166_2.NO2
- new net VEXT: SPLY-EXT.2, TS5A4624.NO, VMCU_EXT.A
- new net VOUT: TS5A3159.COM
- new net V_CALIB: TS5A23166_1.IN1, TS5A23166_1.IN2, TS5A23166_2.IN1, TS5A23166_2.IN2, TS5A3159.NC, VCALIB_LED.A
- net -12OUT: now also L1.1; no longer U$1.1
- net 5V5: now also D1.C, REG.EN, REG.VIN, REG.VIN_2; no longer CR3.12, U3.EN, U3.VIN, U3.VIN_2
- net 5VR: now also +-12V.VIN1, +-12V.VIN2, C10.1, L3.1, L4.1, R20.2, R21.2, R22.2, R23.2, REG.SENSE, REG.VOUT, REG.VOUT_2, TS5A23166_1.V+, TS5A23166_2.V+; no longer U3.SENSE, U3.VOUT, U3.VOUT_2
- net 5VUSB: now also BOOST.EN, BOOST.VIN, C23.1, L2.1, L5.2; no longer J1.VBUS, U$9.1, U4.EN, U4.VIN
- net DGND: now also R31.1, R32.1, R33.2, R34.2, R35.1, R36.2, R45.1, R46.1, R47.1, R48.1, R49.1, R50.1, R51.1, R52.1, R53.1, TS5A23166_1.GND, TS5A23166_2.GND, TS5A3159.GND; no longer R31.2, R32.2
- net FB: now also BOOST.FB, R27.2; no longer U4.FB
- net GND: now also BOOST.PGND, C22.2, C23.2, D3.C, R36.1, REG.EP, REG.GND, SPLY-EXT.1; no longer CR2.12, U3.EP, U3.GND, U4.PGND
- net N$13: now also D2.C; no longer CR1.12
- net N$14: now also D3.A, L1.2; no longer CR2.21, U$1.2
- net N$20: now also REG.SS; no longer U3.SS
- net SW: now also BOOST.SW, D1.A, L2.2; no longer CR3.21, U$9.2, U4.SW
- net SWB1: now also D2.A; no longer CR1.21
- net SW_CTRL_PWR: now also CTRL.2, R51.2
- net VC1: now also +-12V.VC1
- net VSPLY: now also AD8422.IN+, R1.1, U$1.I1; no longer U$6.I1
- net VSS: now also TS5A3159.NO, U$1.I2, VMCU_LED.A; no longer U$6.I2
Other:
- note added: "5V boost to 5.5V"
- note added: "Missing input SW_CTRL_PWR"
- note added: "UTILITY PINS"
- note removed: "USB ~5V boost to 5.5V"
- moved on the sheet: C17, C18, C19, C20, C21, J1, MCU_VUSB, R27, R28, R29, R30, SEL-SPLY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

Commit message: add usb ports to schematics
Parts:
- added ADC: 455-1750-1-ND, SparkFun-Connectors:CONN_03
- added TP1, TP2: TEST-POINT3, SparkFun-Connectors:TEST-POINT3
- J1: value USB_A_SMT_FEMALE -> 10118194-0001LF; device SparkFun-Connectors:USB_A_SMT_FEMALE -> 10118194-0001LF:10118194-0001LF
- MCU: value (none) -> USB_A_SMT_FEMALE; device SparkFun-Connectors:CONN_02 -> SparkFun-Connectors:USB_A_SMT_FEMALE
Connections:
- net N$15 renamed D+
- net N$16 renamed D-
- removed net N$11: AD8422.VOUT, R15.1
- removed net N$18: AD8629-4.OUT, R12.1, R13.2
- new net SHUNT+: AD8422.IN+, R1.1, U$1.E1
- new net SHUNT-: AD8422.IN-, R5.1, U$1.E2
- new net VHOUT: AD8422.VOUT, ADC.3, R15.1
- new net VLOUT: AD8629-4.OUT, ADC.2, R12.1, R13.2
- net 5VIN: no longer J1.VBUS
- net 5VUSB: now also J1.VDD
- net DGND: now also J1.GND
- net GND: now also ADC.1, MCU.GND; no longer J1.GND, MCU.1
- net STG1: now also TP1.1
- net VSPLY: no longer AD8422.IN+, R1.1
- net VSS: now also MCU.VBUS, TP2.1; no longer AD8422.IN-, MCU.2, R5.1
Other:
- note added: "MICRO USB"
- moved on the sheet: +-12V, C10, C11, C15, C16, C9, J1, L3, L4, R18, R19, R20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
