File: v0.2/board/cm_ADA4522.sch (EAGLE design)
At the start: 109 parts, among them J1 10118194-0001LF

Commit message: change AD8629 to ADA4522
Parts:
- removed AD8629-1, AD8629-2, AD8629-3, AD8629-4: AD8629, SparkFun-IC-Amplifiers:AD8629
- removed CALIB-RES: (no value), pinhead:PINHD-1X4
- removed CTRL: (no value), pinhead:PINHD-1X2
- removed POWER: (no value), SparkFun-Connectors:CONN_05
- removed SEL-SPLY1: (no value), SparkFun-Connectors:CONN_02
- added C24: 100n, SparkFun-Capacitors:10UF-0603-6.3V-20%
- added J2: (no value), SparkFun-Connectors:CONN_06LONGPADS
- added J3: (no value), SparkFun-Connectors:CONN_04
- added U1: ADA4522-4ARZ, ADA4522-4:ADA4522-4ARZ
- R12: value 2k -> 10k
- R6, R7: value 100 -> 1k
Connections:
- removed net N$1: AD8629-2.+IN, C2.1, C3.2, R5.2
- removed net N$17: AD8629-4.-IN, R11.2, R12.2
- removed net N$2: AD8629-1.OUT, R2.1, R6.1
- removed net N$3: AD8629-1.-IN, R2.2, R3.1
- removed net N$4: AD8629-2.-IN, R3.2, R4.1
- removed net N$5: AD8629-2.OUT, R4.2, R7.1
- removed net N$6: AD8629-1.+IN, C1.2, C3.1, R1.2
- removed net N$8: AD8629-3.-IN, R6.2, R8.1
- removed net N$9: AD8629-3.+IN, R7.2, R9.1
- removed net STG1: AD8629-3.OUT, AD8629-4.+IN, R10.2, R8.2, TP1.1
- removed net VDD: AD8629-1.V+, AD8629-2.V+, AD8629-3.V+, AD8629-4.V+, C4.1, C5.1, C6.1, C7.1, POWER.3, SEL-SPLY1.2
- new net +IN_A: C1.2, C3.1, R1.2, U1.+IN_A
- new net +IN_B: C2.1, C3.2, R5.2, U1.+IN_B
- new net +IN_C: R6.2, R8.1, U1.+IN_C
- new net -IN_A: R2.2, R3.1, U1.-IN_A
- new net -IN_B: R3.2, R4.1, U1.-IN_B
- new net -IN_C: R11.2, R12.2, R7.2, R9.1, U1.-IN_C
- new net -IN_D: U1.-IN_D
- new net OUT_A: R2.1, R6.1, U1.OUT_A
- new net OUT_B: R4.2, R7.1, U1.OUT_B
- new net OUT_C: R10.2, R8.2, TP1.1, U1.+IN_D, U1.OUT_C
- new net OUT_D: R12.1, R13.2
- net +12V: now also C4.1, C5.1, J3.4, U1.V+; no longer POWER.5
- net -12V: now also C6.1, C7.1, J3.3, U1.V-; no longer POWER.4
- net 5V5: no longer SEL-SPLY1.1
- net 5VIN: now also J1.VDD
- net 5VUSB: now also C24.1; no longer J1.VDD
- net GND: now also C24.2, J3.1; no longer AD8629-1.V-, AD8629-2.V-, AD8629-3.V-, AD8629-4.V-, POWER.1
- net SW_CTRL_0: now also J2.2; no longer CTRL.1
- net SW_CTRL_1: now also J2.3; no longer CALIB-RES.1
- net SW_CTRL_2: now also J2.4; no longer CALIB-RES.2
- net SW_CTRL_3: now also J2.5; no longer CALIB-RES.3
- net SW_CTRL_4: now also J2.6; no longer CALIB-RES.4
- net SW_CTRL_PWR: now also J2.1; no longer CTRL.2
- net VLOUT: now also U1.OUT_D; no longer AD8629-4.OUT, R12.1, R13.2
- net VSPLY: now also J3.2; no longer POWER.2
Other:
- note removed: "Missing input SW_CTRL_PWR"
- moved on the sheet: C2, C3, R10, R11, R12, R13, R2, R3, R4, R5, R6, R7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

Commit message: connect data ports from usb
Connections:
- removed net D+: J1.D+
- removed net D-: J1.D-
- new net DATA+: J1.D+, MCU.D+
- new net DATA-: J1.D-, MCU.D-
Changed lines of the file:
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@@
+</segment>
+</net>
+<net name="DATA+" class="0">
+<segment>
+<pinref part="MCU" gate="G$1" pin="D+"/>
+<wire x1="154.94" y1="-86.36" x2="160.02" y2="-86.36" width="0.1524" layer="91"/>
+</segment>
+</net>
+<net name="DATA-" class="0">
+<segment>
+<pinref part="MCU" gate="G$1" pin="D-"/>
+<wire x1="160.02" y1="-88.9" x2="154.94" y2="-88.9" width="0.1524" layer="91"/>
 </segment>
 </net>
@@
 </segment>
 </net>
-<net name="D-" class="0">
+<net name="DATA-" class="0">
 <segment>
 <pinref part="J1" gate="G$1" pin="D-"/>
@@
 </segment>
 </net>
-<net name="D+" class="0">
+<net name="DATA+" class="0">
 <segment>
 <pinref part="J1" gate="G$1" pin="D+"/>

Commit message: add names to external connectors
Parts:
- renumbered J1 to USB-IN, J2 to SWITCH, J3 to POWER, MCU to USB-OUT, MCU_VUSB to VUSB, VCALIB_LED to CALIB, VMCU_EXT to VEXT, VMCU_LED to VMCU
