File: v0.2/boards/cm_ltc6102_L/cm_ltc6102.sch (EAGLE design)
At the start: 98 parts, among them J1 10118194-0001LF, U1 ADA4528-2ARMZ-R7, U10 TS5A3159ADBVRDBV6-M, U2 LTC6102IMS8PBF, U3 ADM7170ACPZ-1.3-R7CP_8_21-M, U4 MIC2250-1YD5TSOT-23-5_D5-M, U6 TS3A4751PWRPW14-M, U7 TS5A4624DCKRDCK6-M, X1 PN87520-S

Commit message: cm_ltc6102_L: modify layout, finish silkscreen
Parts:
- renumbered JP4 to JP2, U1 to ADA4528, U10 to TS5A3159, U3 to ADM7170, U4 to MIC2250, U6 to TS3A4651, U7 to TS5A4624, VMCU_LED1 to VMCU_EXT_LED
Connections:
- net ALERT: now also JP2.4; no longer JP2.2
- net SCL: now also JP2.2; no longer JP2.4

Commit message: cm_ltc6102_L: fix wrong sized ic and surface capacitor
Parts:
- removed C12: 10uF x7R, rcl:C-EUC0603
- removed TS3A4651: TS3A4751PWRPW14-M, texas_instruments:TS3A4751PWRPW14-M
- added C11: 10uF x7R, rcl:C-EUC0805
- added TS5A23166_1, TS5A23166_2: TS5A23166DCURDCU8-M, texas_instruments:TS5A23166DCURDCU8-M
- C8: device rcl:C-EUC0603 -> rcl:C-EUC0805
- R12: value 100k 0.01% -> 100k 0.05%
Connections:
- net 5V_F: now also C8.1, TS5A23166_1.V+, TS5A23166_2.V+; no longer C12.1, TS3A4651.V+
- net DGND: now also TS5A23166_1.GND, TS5A23166_2.GND; no longer TS3A4651.GND
- net GND: now also C11.2; no longer C12.2
- net LTC_VCC: now also C11.1; no longer C8.1
- net N$30: now also TS5A23166_1.COM1; no longer TS3A4651.NO1
- net N$31: now also TS5A23166_1.COM2; no longer TS3A4651.NO2
- net N$32: now also TS5A23166_2.COM1; no longer TS3A4651.NO3
- net N$33: now also TS5A23166_2.COM2; no longer TS3A4651.NO4
- net SW_CTRL_1: now also TS5A23166_1.NO1; no longer TS3A4651.IN1
- net SW_CTRL_2: now also TS5A23166_1.NO2; no longer TS3A4651.IN2
- net SW_CTRL_3: now also TS5A23166_2.NO1; no longer TS3A4651.IN3
- net SW_CTRL_4: now also TS5A23166_2.NO2; no longer TS3A4651.IN4
- net V_CALIB: now also TS5A23166_1.IN1, TS5A23166_1.IN2, TS5A23166_2.IN1, TS5A23166_2.IN2; no longer TS3A4651.COM1, TS3A4651.COM2, TS3A4651.COM3, TS3A4651.COM4
Other:
- moved on the sheet: C8, R23, R24, R25, R26

Commit message: fix enable pull ups error, update bom
Parts:
- removed R17, R4, R9: 10k 1%, resistor:R-EU_R0603
Connections:
- removed net N$15: ADM7170.EN, R4.2
- removed net N$18: MIC2250.EN, R17.1
- removed net N$5: R9.2, U2.V-/EN
- net 5.5V: now also ADM7170.EN; no longer R4.1
- net 5V_F: now also MIC2250.EN; no longer R17.2
- net GND: now also U2.V-/EN
- net LTC_VCC: no longer R9.1
Changed lines of the file:
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@@
 <part name="U$1" library="vishay" deviceset="VCS1625Z" device=""/>
 <part name="GND1" library="supply1" library_urn="urn:adsk.eagle:library:371" deviceset="GND" device=""/>
-<part name="R9" library="resistor" library_urn="urn:adsk.eagle:library:348" deviceset="R-EU_" device="R0603" package3d_urn="urn:adsk.eagle:package:26057/1" value="10k 1%"/>
 <part name="R10" library="resistor" library_urn="urn:adsk.eagle:library:348" deviceset="R-EU_" device="R0603" package3d_urn="urn:adsk.eagle:package:26057/1" value="10k 0.01%"/>
 <part name="GND2" library="supply1" library_urn="urn:adsk.eagle:library:371" deviceset="GND" device=""/>
@@
 <part name="GND14" library="supply1" library_urn="urn:adsk.eagle:library:371" deviceset="GND" device=""/>
 <part name="GND15" library="supply1" library_urn="urn:adsk.eagle:library:371" deviceset="GND" device=""/>
-<part name="R4" library="resistor" library_urn="urn:adsk.eagle:library:348" deviceset="R-EU_" device="R0603" package3d_urn="urn:adsk.eagle:package:26057/1" value="10k 1%"/>
 <part name="MIC2250" library="texas_instruments" deviceset="MIC2250-1YD5" device="TSOT-23-5_D5-M"/>
 <part name="R15" library="rcl" library_urn="urn:adsk.eagle:library:334" deviceset="R-US_" device="R0603" package3d_urn="urn:adsk.eagle:package:23555/1" value="100k 1%"/>
 <part name="R16" library="rcl" library_urn="urn:adsk.eagle:library:334" deviceset="R-US_" device="R0603" package3d_urn="urn:adsk.eagle:package:23555/1" value="29K 1%"/>
-<part name="R17" library="resistor" library_urn="urn:adsk.eagle:library:348" deviceset="R-EU_" device="R0603" package3d_urn="urn:adsk.eagle:package:26057/1" value="10k 1%"/>
 <part name="C13" library="rcl" library_urn="urn:adsk.eagle:library:334" deviceset="C-EU" device="C0603" package3d_urn="urn:adsk.eagle:package:23616/1" value="2.2uF"/>
 <part name="D1" library="diode" library_urn="urn:adsk.eagle:library:210" deviceset="DIODE-" device="SOD80C"/>
@@
 <part name="C11" library="rcl" library_urn="urn:adsk.eagle:library:334" deviceset="C-EU" device="C0805" package3d_urn="urn:adsk.eagle:package:23617/1" value="10uF x7R"/>
 <part name="C8" library="rcl" library_urn="urn:adsk.eagle:library:334" deviceset="C-EU" device="C0805" package3d_urn="urn:adsk.eagle:package:23617/1" value="10uF x7R"/>
+<part name="GND17" library="supply1" library_urn="urn:adsk.eagle:library:371" deviceset="GND" device=""/>
 </parts>
 <sheets>
@@
 <instance part="U$1" gate="A" x="88.9" y="370.84" rot="R90"/>
 <instance part="GND1" gate="1" x="132.08" y="403.86"/>
-<instance part="R9" gate="G$1" x="53.34" y="431.8" rot="R270"/>
 <instance part="R10" gate="G$1" x="248.92" y="421.64" rot="R90"/>
 <instance part="GND2" gate="1" x="248.92" y="414.02"/>
@@
 <instance part="GND14" gate="1" x="-134.62" y="55.88"/>
 <instance part="GND15" gate="1" x="-144.78" y="55.88"/>
-<instance part="R4" gate="G$1" x="-228.6" y="81.28"/>
 <instance part="MIC2250" gate="A" x="-99.06" y="154.94"/>
 <instance part="R15" gate="G$1" x="-121.92" y="139.7" rot="R180"/>
 <instance part="R16" gate="G$1" x="-116.84" y="127" rot="R270"/>
-<instance part="R17" gate="G$1" x="-55.88" y="137.16" rot="R270"/>
 <instance part="C13" gate="G$1" x="-127" y="124.46" rot="R180"/>
 <instance part="D1" gate="G$1" x="-109.22" y="154.94" rot="R180"/>
@@
 <instance part="C11" gate="G$1" x="-144.78" y="320.04"/>
 <instance part="C8" gate="G$1" x="-48.26" y="129.54"/>
+<instance part="GND17" gate="1" x="35.56" y="408.94"/>
 </instances>
 <busses>
@@
 </segment>
 <segment>
-<pinref part="R9" gate="G$1" pin="1"/>
-<wire x1="53.34" y1="436.88" x2="53.34" y2="441.96" width="0.1524" layer="91"/>
-<label x="53.34" y="444.5" size="1.778" layer="95" rot="R90"/>
-</segment>
-<segment>
 <wire x1="-144.78" y1="322.58" x2="-144.78" y2="327.66" width="0.1524" layer="91"/>
 <pinref part="R14" gate="G$1" pin="1"/>
@@
 <pinref part="GND30" gate="1" pin="GND"/>
 </segment>
+<segment>
+<pinref part="U2" gate="A" pin="V-/EN"/>
+<wire x1="71.12" y1="416.56" x2="35.56" y2="416.56" width="0.1524" layer="91"/>
+<wire x1="35.56" y1="416.56" x2="35.56" y2="411.48" width="0.1524" layer="91"/>
+<pinref part="GND17" gate="1" pin="GND"/>
+</segment>
 </net>
 <net name="VOUT" class="0">
@@
 <label x="-190.5" y="365.76" size="1.778" layer="95"/>
 <wire x1="-200.66" y1="365.76" x2="-193.04" y2="365.76" width="0.1524" layer="91"/>
-</segment>
-</net>
-<net name="N$5" class="0">
-<segment>
-<pinref part="U2" gate="A" pin="V-/EN"/>
-<pinref part="R9" gate="G$1" pin="2"/>
-<wire x1="53.34" y1="426.72" x2="53.34" y2="416.56" width="0.1524" layer="91"/>
-<wire x1="53.34" y1="416.56" x2="71.12" y2="416.56" width="0.1524" layer="91"/>
 </segment>
 </net>
@@
 </segment>
 </net>
-<net name="N$15" class="0">
-<segment>
-<pinref part="ADM7170" gate="A" pin="EN"/>
-<wire x1="-220.98" y1="81.28" x2="-228.6" y2="81.28" width="0.1524" layer="91"/>
-<wire x1="-226.06" y1="81.28" x2="-223.52" y2="81.28" width="0.1524" layer="91"/>
-<pinref part="R4" gate="G$1" pin="2"/>
-</segment>
-</net>
 <net name="N$10" class="0">
 <segment>
@@
 </segment>
 </net>
-<net name="N$18" class="0">
-<segment>
-<pinref part="MIC2250" gate="A" pin="EN"/>
-<wire x1="-60.96" y1="152.4" x2="-55.88" y2="152.4" width="0.1524" layer="91"/>
-<wire x1="-55.88" y1="152.4" x2="-55.88" y2="142.24" width="0.1524" layer="91"/>
-<pinref part="R17" gate="G$1" pin="1"/>
-</segment>
-</net>
 <net name="5.5V" class="0">
 <segment>
 <pinref part="ADM7170" gate="A" pin="VIN_2"/>
-<wire x1="-220.98" y1="96.52" x2="-269.24" y2="96.52" width="0.1524" layer="91"/>
+<wire x1="-220.98" y1="96.52" x2="-236.22" y2="96.52" width="0.1524" layer="91"/>
+<wire x1="-236.22" y1="96.52" x2="-269.24" y2="96.52" width="0.1524" layer="91"/>
 <wire x1="-269.24" y1="96.52" x2="-269.24" y2="93.98" width="0.1524" layer="91"/>
 <pinref part="ADM7170" gate="A" pin="VIN"/>
@@
 <label x="-269.24" y="111.76" size="1.778" layer="95" rot="R90"/>
 <wire x1="-269.24" y1="96.52" x2="-269.24" y2="109.22" width="0.1524" layer="91"/>
-</segment>
-<segment>
-<pinref part="R4" gate="G$1" pin="1"/>
-<wire x1="-233.68" y1="81.28" x2="-236.22" y2="81.28" width="0.1524" layer="91"/>
-<label x="-241.3" y="81.28" size="1.778" layer="95"/>
+<pinref part="ADM7170" gate="A" pin="EN"/>
+<wire x1="-220.98" y1="81.28" x2="-236.22" y2="81.28" width="0.1524" layer="91"/>
+<wire x1="-236.22" y1="81.28" x2="-236.22" y2="96.52" width="0.1524" layer="91"/>
+<junction x="-236.22" y="96.52"/>
 </segment>
 <segment>
@@
 <wire x1="-58.42" y1="170.18" x2="-58.42" y2="154.94" width="0.1524" layer="91"/>
 <pinref part="MIC2250" gate="A" pin="VIN"/>
-<wire x1="-58.42" y1="154.94" x2="-60.96" y2="154.94" width="0.1524" layer="91"/>
-<wire x1="-60.96" y1="154.94" x2="-48.26" y2="154.94" width="0.1524" layer="91"/>
+<wire x1="-60.96" y1="154.94" x2="-58.42" y2="154.94" width="0.1524" layer="91"/>
+<wire x1="-58.42" y1="154.94" x2="-48.26" y2="154.94" width="0.1524" layer="91"/>
 <wire x1="-48.26" y1="154.94" x2="-48.26" y2="132.08" width="0.1524" layer="91"/>
 <label x="-48.26" y="177.8" size="1.778" layer="95" rot="R90"/>
@@
 <junction x="-72.39" y="170.18"/>
 <pinref part="C8" gate="G$1" pin="1"/>
-</segment>
-<segment>
-<pinref part="R17" gate="G$1" pin="2"/>
-<label x="-68.58" y="127" size="1.778" layer="95"/>
-<wire x1="-55.88" y1="132.08" x2="-55.88" y2="127" width="0.1524" layer="91"/>
-<wire x1="-55.88" y1="127" x2="-66.04" y2="127" width="0.1524" layer="91"/>
-</segment>
-<segment>
+<pinref part="MIC2250" gate="A" pin="EN"/>
+<wire x1="-60.96" y1="152.4" x2="-58.42" y2="152.4" width="0.1524" layer="91"/>
+<wire x1="-58.42" y1="152.4" x2="-58.42" y2="154.94" width="0.1524" layer="91"/>
+<junction x="-58.42" y="154.94"/>
+</segment>
+<segment>

Commit message: cm_ltc6102: increase track size add doc
Parts:
- C1: value 0.1uF X7R -> 100nF x7R; device rcl:C-EUC0805 -> rcl:C-EUC0603
- C10, C9: device rcl:C-USC1206 -> rcl:C-EUC1206
Connections:
- net LTC_VCC: now also C1.1; no longer C1.2
- net N$6: now also C1.2; no longer C1.1
Other:
- note added: "ALL SWITCH ARE PD FOR DEFAULT NORMAL OPERATION"
- note added: "CALIBRATION"
- note added: "CALIBRATION RESISTOR DIGITAL SWITCH"
- note added: "Current Measurement"
- note added: "DIGITAL SWITCH TO SELECT EXTERNAL OR USB SUPPLY FOR MCU"
- note added: "EXTERN DIGITAL SWITCH TO SELECT CALIBRATION OR NORMAL OPERATION"
- note added: "PWR Inputs"
- note added: "PWR Regulators"
- moved on the sheet: ADA4528, C1, C15, C2, C3, C4, C5, C6, INA226, JP2, JP5, R1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
